File: Krado from Scratch.sch (KiCad schematic (older format))
At the start: 157 parts, among them SW1 SW_Push, U1 ATmega32U4-AU, Y1 16MHz

Commit message: Tracing
Parts:
- added C8: 22pF, Capacitor_SMD:C_0805_2012Metric, symbol Device:C_Small
- added R7: 330, Resistor_SMD:R_0805_2012Metric, symbol Device:R_Small
- C1, C2, C3, C4, C5, C6, C7: footprint Diode_SMD:D_SOD-123 -> Capacitor_SMD:C_0805_2012Metric
- R6: value 10k -> 1k
Connections:
- net D+: now also R4.1, U1.4 (D+)
- net D-: now also R3.1, U1.3 (D-)
- net GND: now also R7.2; no longer SW1.1
- net RST: now reaches R5.2, SW1.2, U1.13 (~RESET)
- net RST: now also C8.1
- new net: C8.2, R7.1, SW1.1
Other:
- moved on the sheet: R5, SW1
Changed lines of the file:
@@
 P 21500 9550
 F 0 "R6" V 21304 9550 50  0000 C CNN
-F 1 "10k" V 21395 9550 50  0000 C CNN
+F 1 "1k" V 21395 9550 50  0000 C CNN
 F 2 "Resistor_SMD:R_0805_2012Metric" H 21500 9550 50  0001 C CNN
 F 3 "~" H 21500 9550 50  0001 C CNN
@@
 F 0 "C3" H 19092 8896 50  0000 L CNN
 F 1 "1uF" H 19092 8805 50  0000 L CNN
-F 2 "Diode_SMD:D_SOD-123" H 19000 8850 50  0001 C CNN
+F 2 "Capacitor_SMD:C_0805_2012Metric" H 19000 8850 50  0001 C CNN
 F 3 "~" H 19000 8850 50  0001 C CNN
 	1    19000 8850
@@
 F 0 "C4" H 19892 12996 50  0000 L CNN
 F 1 "0.1uF" H 19892 12905 50  0000 L CNN
-F 2 "Diode_SMD:D_SOD-123" H 19800 12950 50  0001 C CNN
+F 2 "Capacitor_SMD:C_0805_2012Metric" H 19800 12950 50  0001 C CNN
 F 3 "~" H 19800 12950 50  0001 C CNN
 	1    19800 12950
@@
 F 0 "C5" H 20392 12996 50  0000 L CNN
 F 1 "0.1uF" H 20392 12905 50  0000 L CNN
-F 2 "Diode_SMD:D_SOD-123" H 20300 12950 50  0001 C CNN
+F 2 "Capacitor_SMD:C_0805_2012Metric" H 20300 12950 50  0001 C CNN
 F 3 "~" H 20300 12950 50  0001 C CNN
 	1    20300 12950
@@
 F 0 "C6" H 20842 12996 50  0000 L CNN
 F 1 "0.1uF" H 20842 12905 50  0000 L CNN
-F 2 "Diode_SMD:D_SOD-123" H 20750 12950 50  0001 C CNN
+F 2 "Capacitor_SMD:C_0805_2012Metric" H 20750 12950 50  0001 C CNN
 F 3 "~" H 20750 12950 50  0001 C CNN
 	1    20750 12950
@@
 F 0 "C7" H 21292 12996 50  0000 L CNN
 F 1 "10uF" H 21292 12905 50  0000 L CNN
-F 2 "Diode_SMD:D_SOD-123" H 21200 12950 50  0001 C CNN
+F 2 "Capacitor_SMD:C_0805_2012Metric" H 21200 12950 50  0001 C CNN
 F 3 "~" H 21200 12950 50  0001 C CNN
 	1    21200 12950
@@
 F 0 "C1" V 18571 7600 50  0000 C CNN
 F 1 "22pF" V 18662 7600 50  0000 C CNN
-F 2 "Diode_SMD:D_SOD-123" H 18800 7600 50  0001 C CNN
+F 2 "Capacitor_SMD:C_0805_2012Metric" H 18800 7600 50  0001 C CNN
 F 3 "~" H 18800 7600 50  0001 C CNN
 	1    18800 7600
@@
 F 0 "C2" V 18571 7950 50  0000 C CNN
 F 1 "22pF" V 18662 7950 50  0000 C CNN
-F 2 "Diode_SMD:D_SOD-123" H 18800 7950 50  0001 C CNN
+F 2 "Capacitor_SMD:C_0805_2012Metric" H 18800 7950 50  0001 C CNN
 F 3 "~" H 18800 7950 50  0001 C CNN
 	1    18800 7950
@@
 L Switch:SW_Push SW1
 U 1 1 60753B4A
-P 19450 7450
-F 0 "SW1" H 19450 7735 50  0000 C CNN
-F 1 "SW_Push" H 19450 7644 50  0000 C CNN
-F 2 "random-keyboard-parts:SKQG-1155865" H 19450 7650 50  0001 C CNN
-F 3 "~" H 19450 7650 50  0001 C CNN
-	1    19450 7450
-	1    0    0    -1
+P 19200 6550
+F 0 "SW1" H 19200 6835 50  0000 C CNN
+F 1 "SW_Push" H 19200 6744 50  0000 C CNN
+F 2 "random-keyboard-parts:SKQG-1155865" H 19200 6750 50  0001 C CNN
+F 3 "~" H 19200 6750 50  0001 C CNN
+	1    19200 6550
+	0    -1   -1   0
 $EndComp
 $Comp
@@
 Wire Wire Line
 	19050 7450 19250 7450
-Wire Wire Line
-	19650 7450 19750 7450
-Wire Wire Line
-	19750 7450 19750 7150
-Connection ~ 19750 7450
-Wire Wire Line
-	19750 7450 19850 7450
-$Comp
-L Device:R_Small R5
-U 1 1 60759043
-P 19750 7050
-F 0 "R5" H 19809 7096 50  0000 L CNN
-F 1 "10k" H 19809 7005 50  0000 L CNN
-F 2 "Resistor_SMD:R_0805_2012Metric" H 19750 7050 50  0001 C CNN
-F 3 "~" H 19750 7050 50  0001 C CNN
-	1    19750 7050
-	1    0    0    -1
-$EndComp
 $Comp
 L power:+5V #PWR0110
 U 1 1 6075A732
-P 19750 6850
-F 0 "#PWR0110" H 19750 6700 50  0001 C CNN
-F 1 "+5V" H 19765 7023 50  0000 C CNN
-F 2 "" H 19750 6850 50  0001 C CNN
-F 3 "" H 19750 6850 50  0001 C CNN
-	1    19750 6850
-	1    0    0    -1
-$EndComp
-Wire Wire Line
-	19750 6950 19750 6850
+P 19300 5900
+F 0 "#PWR0110" H 19300 5750 50  0001 C CNN
+F 1 "+5V" H 19315 6073 50  0000 C CNN
+F 2 "" H 19300 5900 50  0001 C CNN
+F 3 "" H 19300 5900 50  0001 C CNN
+	1    19300 5900
+	1    0    0    -1
+$EndComp
 Text GLabel 18400 8450 0    50   Input ~ 0
 D+
@@
 Text GLabel 21050 10050 2    50   Input ~ 0
 COL15
+Text GLabel 19850 7450 0    50   Input ~ 0
+RST
+Text GLabel 19600 6350 2    50   Input ~ 0
+RST
+$Comp
+L Device:R_Small R7
+U 1 1 60884077
+P 19300 6900
+F 0 "R7" H 19359 6946 50  0000 L CNN
+F 1 "330" H 19359 6855 50  0000 L CNN
+F 2 "Resistor_SMD:R_0805_2012Metric" H 19300 6900 50  0001 C CNN
+F 3 "~" H 19300 6900 50  0001 C CNN
+	1    19300 6900
+	1    0    0    -1
+$EndComp
+Wire Wire Line
+	19200 6750 19200 6800
+Wire Wire Line
+	19200 6800 19300 6800
+$Comp
+L Device:C_Small C8
+U 1 1 608A6977
+P 19450 6550
+F 0 "C8" H 19542 6596 50  0000 L CNN
+F 1 "22pF" H 19542 6505 50  0000 L CNN
+F 2 "Capacitor_SMD:C_0805_2012Metric" H 19450 6550 50  0001 C CNN
+F 3 "~" H 19450 6550 50  0001 C CNN
+	1    19450 6550
+	1    0    0    -1
+$EndComp
+Wire Wire Line
+	19450 6450 19450 6350
+Connection ~ 19450 6350
+Wire Wire Line
+	19450 6350 19600 6350
+Wire Wire Line
+	19450 6650 19450 6800
+Wire Wire Line
+	19450 6800 19300 6800
+Connection ~ 19300 6800
+$Comp
+L power:GND #PWR0114
+U 1 1 608E730E
+P 19300 7150
+F 0 "#PWR0114" H 19300 6900 50  0001 C CNN
+F 1 "GND" H 19305 6977 50  0000 C CNN
+F 2 "" H 19300 7150 50  0001 C CNN
+F 3 "" H 19300 7150 50  0001 C CNN
+	1    19300 7150
+	1    0    0    -1
+$EndComp
+Wire Wire Line
+	19300 7150 19300 7000
+Wire Wire Line
+	19300 5900 19300 6000
+Wire Wire Line
+	19200 6350 19300 6350
+$Comp
+L Device:R_Small R5
+U 1 1 60759043
+P 19300 6100
+F 0 "R5" H 19359 6146 50  0000 L CNN
+F 1 "10k" H 19359 6055 50  0000 L CNN
+F 2 "Resistor_SMD:R_0805_2012Metric" H 19300 6100 50  0001 C CNN
+F 3 "~" H 19300 6100 50  0001 C CNN
+	1    19300 6100
+	1    0    0    -1
+$EndComp
+Wire Wire Line
+	19300 6200 19300 6350
+Connection ~ 19300 6350
+Wire Wire Line
+	19300 6350 19450 6350
+Text Label 19550 8450 0    50   ~ 0
+D+
+Text Label 19300 8550 0    50   ~ 0
+D-
 $EndSCHEMATC
