File: Krado from Scratch.sch (KiCad schematic (older format))
At the start: 159 parts, among them SW1 SW_Push, U1 ATmega32U4-AU, Y1 16MHz

Commit message: Renamed Ref
Parts:
- added U2: PRTR5V0U2X, random-keyboard-parts:SOT143B, symbol random-keyboard-parts:PRTR5V0U2X
- K01: renamed from KY_ESC1; value MX-NoLED -> ESC
- K02: renamed from KY_GRAVE1; value MX-NoLED -> ~`
- K03: renamed from KY_1; value MX-NoLED -> 1!
- K04: renamed from KY_2; value MX-NoLED -> 2@
- K05: renamed from KY_3; value MX-NoLED -> 3#
- K06: renamed from KY_4; value MX-NoLED -> 4$
- K07: renamed from KY_5; value MX-NoLED -> 5%
- K08: renamed from KY_6; value MX-NoLED -> 6^
- K09: renamed from KY_7; value MX-NoLED -> 7&
- K10: renamed from KY_8; value MX-NoLED -> 8*
- K11: renamed from KY_9; value MX-NoLED -> 9(
- K12: renamed from KY_0; value MX-NoLED -> 0)
- K13: renamed from KY_MINUS1; value MX-NoLED -> -_
- K14: renamed from KY_EQUALS1; value MX-NoLED -> =
- K15: renamed from BACKSPLIT1; value MX-NoLED -> BACKSPLIT1
- K16: renamed from BACKSPLIT2; value MX-NoLED -> BACKSPLIT2
- K18: renamed from 2U_BACKSPACE1; value MX-NoLED -> 2U_BACKSPACE
- K19: renamed from MOD_TAB1; value MX-NoLED -> TAB
- K20: renamed from KY_Q1; value MX-NoLED -> Q
- K21: renamed from KY_W1; value MX-NoLED -> W
- K22: renamed from KY_E1; value MX-NoLED -> E
- K23: renamed from KY_R1; value MX-NoLED -> R
- K24: renamed from KY_T1; value MX-NoLED -> T
- K25: renamed from KY_Y1; value MX-NoLED -> Y
- K26: renamed from KY_U1; value MX-NoLED -> U
- K27: renamed from KY_I1; value MX-NoLED -> I
- K28: renamed from KY_O1; value MX-NoLED -> O
- K29: renamed from KY_P1; value MX-NoLED -> P
- K30: renamed from KY_LBRACK1; value MX-NoLED -> [{
- K31: renamed from KY_RBRACK1; value MX-NoLED -> }]
- K32: renamed from KY_BAR1; value MX-NoLED -> BAR-BACKSLASH
- K33: renamed from STEPPED_CAPS1; value MX-NoLED -> STEP_CAPS
- K34: renamed from MOD_CAPS1; value MX-NoLED -> CAPS
- K35: renamed from KY_A1; value MX-NoLED -> A
- K36: renamed from KY_S1; value MX-NoLED -> S
- K37: renamed from KY_D1; value MX-NoLED -> D
- K38: renamed from KY_F1; value MX-NoLED -> F
- K39: renamed from KY_G1; value MX-NoLED -> G
- K40: renamed from KY_H1; value MX-NoLED -> H
- K41: renamed from KY_J1; value MX-NoLED -> J
- K42: renamed from KY_K1; value MX-NoLED -> K
- K43: renamed from KY_L1; value MX-NoLED -> L
- K44: renamed from KY_COLON1; value MX-NoLED -> COLON
- K45: renamed from KY_QUOTE1; value MX-NoLED -> '\"
- K46: renamed from MOD_ENTER1; value MX-NoLED -> ENTER
- K47: renamed from MOD_L_SHIFT1; value MX-NoLED -> L_SHIFT
- K48: renamed from KY_Z1; value MX-NoLED -> Z
- K49: renamed from KY_X1; value MX-NoLED -> X
- K50: renamed from KY_C1; value MX-NoLED -> C
- K51: renamed from KY_V1; value MX-NoLED -> V
- K52: renamed from KY_B1; value MX-NoLED -> B
- K53: renamed from KY_N1; value MX-NoLED -> N
- K54: renamed from KY_M1; value MX-NoLED -> M
- K55: renamed from KY_COMMA1; value MX-NoLED -> COMMA
- K56: renamed from KY_PERIOD1; value MX-NoLED -> .>
- K57: renamed from KY_QUESTION1; value MX-NoLED -> /?
- K58: renamed from MOD_R_SHIFT1; value MX-NoLED -> R_SHIFT_1.75U
- K59: renamed from 2.75U_SHIFT1; value MX-NoLED -> R_SHIFT_2.75
- K60: renamed from UPARROW1; value MX-NoLED -> UP
- K61: renamed from FN1; value MX-NoLED -> FN1
- K62: renamed from L_CTRL1; value MX-NoLED -> L_CTRL
- K63: renamed from L_GUI1; value MX-NoLED -> L_GUI
- K64: renamed from L_ALT1; value MX-NoLED -> L_ALT
- K65: renamed from SPACE1; value MX-NoLED -> SPACE
- K66: renamed from 1U_R_ALT1; value MX-NoLED -> 1U_R_ALT1
- K67: renamed from 1.25U_R_ALT1; value MX-NoLED -> 1.25U_R_ALT1
- K68: renamed from 1U_PN1; value MX-NoLED -> 1U_PN1
- K69: renamed from 1.25U_PN2; value MX-NoLED -> 1.25U_PN2
- K70: renamed from R_CTRL1; value MX-NoLED -> R_CTRL
- K71: renamed from LEFTARROW1; value MX-NoLED -> LEFT
- K72: renamed from DOWNARROW1; value MX-NoLED -> DOWNARROW
- K73: renamed from RIGHTARROW1; value MX-NoLED -> RIGHT
- R6: value 1k -> 10k
Connections:
- net D+: now also U2.2 (IO1)
- net D-: now also U2.3 (IO2)
- net GND: now also U2.1 (GND)
- net VCC: now also U2.4 (VCC)
- no-connect marks 0 -> 3
Other:
- moved on the sheet: F1, R1, R2, USB1
