File: Krado from Scratch.kicad_pcb (KiCad board)
At the start: 2 copper layers, 157 parts, among them SW1 SW_Push, U1 ATmega32U4-AU, Y1 16MHz

Commit message: PCB Switches Layout
Parts:
- KY_BAR1: footprint MX_Only:MXOnly-1U-Hotswap -> MX_Only:MXOnly-1.5U-Hotswap
- moved KY_2 277.3 mm to (81.0, 33.3)
- moved KY_ESC1 254.6 mm to (23.8, 33.3)
- moved D17 250.1 mm to (29.6, 9.55), turned to 90 degrees
- moved KY_A1 242.7 mm to (61.9, 71.4)
- moved D19 242.0 mm to (29.6, 15.3), turned to 90 degrees
- moved KY_F1 238.1 mm to (119.1, 71.4)
- moved D22 232.7 mm to (62.6, -4.65), turned to 90 degrees
- moved D23 232.1 mm to (59.3, -4.65), turned to 90 degrees
- moved D25 231.6 mm to (52.6, -4.95), turned to 90 degrees
- moved C3 231.6 mm to (55.9, -4.65), turned to 90 degrees
- moved KY_5 231.2 mm to (138.1, 33.3)
- moved KY_4 227.7 mm to (119.1, 33.3)
- moved KY_GRAVE1 226.1 mm to (42.9, 33.3)
- moved KY_X1 219.8 mm to (81.0, 90.5)
- moved KY_D1 212.0 mm to (100.0, 71.4)
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- renumbered MOD_TAB2 to MOD_CAPS1

Commit message: PCB Mapped
Parts:
- C1, C2, C3, C4, C5, C6, C7, D1, D10, D11, D12, D13, D14, D15, D16, D17, D18, D19, D2, D20, D21, D22, D23, D24, D25, D26, D27, D28, D29, D3, D30, D31, D32, D33, D34, D35, D36, D37, D38, D39, D4, D40, D41, D42, D43, D44, D45, D46, D47, D48, D49, D5, D50, D51, D52, D53, D54, D55, D56, D57, D58, D59, D6, D60, D61, D62, D63, D64, D66, D67, D7, D8, D9, F1, R1, R2, R3, R4, R5, R6, SW1, U1, USB1, Y1: moved to B.Cu
- moved D4 292.5 mm to (50.0, 51.6), turned to 270 degrees
- moved D5 288.5 mm to (47.6, 71.4), turned to 270 degrees
- moved D14 256.1 mm to (88.9, 52.4), turned to 270 degrees
- moved D52 228.5 mm to (260.4, 33.3), turned to 270 degrees
- moved D2 214.5 mm to (31.8, 109.5), turned to 270 degrees
- moved D6 214.5 mm to (48.4, 90.5), turned to 270 degrees
- moved D1 210.7 mm to (31.8, 33.3), turned to 270 degrees
- moved D53 207.1 mm to (260.4, 52.4), turned to 270 degrees
- moved D65 204.0 mm to (317.5, 29.4)
- moved D3 200.9 mm to (50.8, 33.3), turned to 270 degrees
- moved D59 191.5 mm to (292.9, 71.4), turned to 270 degrees
- moved D31 184.0 mm to (165.1, 52.4), turned to 270 degrees
- moved D32 181.5 mm to (165.1, 71.4), turned to 270 degrees
- moved D43 180.6 mm to (222.2, 52.4), turned to 270 degrees
- moved D30 178.5 mm to (165.1, 33.3), turned to 270 degrees
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Connections:
- U1 pad 10: Net-(U1-Pad10) -> ROW2
- U1 pad 11: Net-(U1-Pad11) -> ROW3
- U1 pad 12: Net-(U1-Pad12) -> COL2
- U1 pad 18: Net-(U1-Pad18) -> COL5
- U1 pad 19: Net-(U1-Pad19) -> COL6
- U1 pad 20: Net-(U1-Pad20) -> COL7
- U1 pad 21: Net-(U1-Pad21) -> COL8
- U1 pad 22: Net-(U1-Pad22) -> COL10
- U1 pad 25: Net-(U1-Pad25) -> COL9
- U1 pad 26: Net-(U1-Pad26) -> COL11
- U1 pad 27: Net-(U1-Pad27) -> COL12
- U1 pad 28: Net-(U1-Pad28) -> ROW4
- U1 pad 29: Net-(U1-Pad29) -> COL0
- U1 pad 30: Net-(U1-Pad30) -> COL1
- U1 pad 31: Net-(U1-Pad31) -> COL3
- U1 pad 32: Net-(U1-Pad32) -> COL4
- U1 pad 39: Net-(U1-Pad39) -> COL15
- U1 pad 40: Net-(U1-Pad40) -> COL14
- U1 pad 41: Net-(U1-Pad41) -> COL13
- U1 pad 8: Net-(U1-Pad8) -> ROW0
- U1 pad 9: Net-(U1-Pad9) -> ROW1

Commit message: PCB Cleaned Up
Parts:
- D65: moved to B.Cu
- moved R4 117.8 mm to (158.8, 121.4)
- moved R3 114.2 mm to (158.8, 117.5)
- moved C7 72.2 mm to (171.4, 129.4), turned to 0 degrees
- moved SPACE1 70.0 mm to (135.7, 179.4)
- moved C4 65.6 mm to (167.5, 114.3)
- moved C1 65.3 mm to (182.6, 107.2), turned to 90 degrees
- moved Y1 64.6 mm to (176.2, 107.2), turned to 180 degrees
- moved U1 64.3 mm to (177.0, 119.9)
- moved C3 62.0 mm to (165.1, 122.2), turned to 0 degrees
- moved C5 53.2 mm to (188.9, 114.3), turned to 90 degrees
- moved C6 50.3 mm to (181.8, 129.4), turned to 180 degrees
- moved C2 49.2 mm to (169.9, 107.2)
- moved R1 44.5 mm to (184.2, 24.6)
- moved R6 39.5 mm to (164.3, 113.5), turned to 90 degrees
- moved R5 37.9 mm to (155.6, 25.4)
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
Commit message: Tracing
Parts:
- added C8: 22pF, Capacitor_SMD:C_0805_2012Metric, B.Cu at (300.8, 65.1)
- added R7: 330, Resistor_SMD:R_0805_2012Metric, B.Cu at (305.2, 65.1)
- C1, C2, C3, C4, C5, C6, C7: footprint Diode_SMD:D_SOD-123 -> Capacitor_SMD:C_0805_2012Metric
- D29: moved to F.Cu
- KY_BAR1: footprint MX_Only:MXOnly-1.5U-Hotswap -> MX_Only:MXOnly-1U-Hotswap
- R6: value 10k -> 1k
- moved D29 70.0 mm to (145.3, 179.4), turned to 270 degrees
- moved C5 29.8 mm to (167.5, 134.9), turned to 0 degrees
- moved C6 29.4 mm to (152.4, 127.8), turned to 90 degrees
- moved C7 22.5 mm to (152.4, 117.5), turned to 270 degrees
- moved C1 22.4 mm to (173.8, 127.8), turned to 0 degrees
- moved R4 16.7 mm to (160.3, 104.8), turned to 270 degrees
- moved U1 15.4 mm to (161.9, 123.0), turned to 270 degrees
- moved Y1 15.1 mm to (176.2, 122.2), turned to 90 degrees
- moved R3 13.9 mm to (164.3, 104.8), turned to 270 degrees
- moved C3 12.4 mm to (159.5, 111.1), turned to 270 degrees
- moved C2 10.3 mm to (173.8, 116.7), turned to 180 degrees
- moved C4 6.40 mm to (173.0, 111.1), turned to 180 degrees
- moved R6 5.08 mm to (168.3, 110.3), turned to 0 degrees
- moved R2 3.97 mm to (188.1, 21.4), turned to 90 degrees
- moved R1 3.97 mm to (181.8, 21.4), turned to 90 degrees
Connections:
- net Net-(R5-Pad2) renamed RST
- R3 pad 1: Net-(R3-Pad1) -> D-
- R4 pad 1: Net-(R4-Pad1) -> D+
- SW1 pad 1: GND -> Net-(C8-Pad2)
- U1 pad 3: Net-(R3-Pad1) -> D-
- U1 pad 4: Net-(R4-Pad1) -> D+
Routing:
- net GND: track 0.00 -> 22.2 mm
- net Net-(C2-Pad1): track 0.00 -> 15.7 mm
- net Net-(C1-Pad1): track 0.00 -> 13.3 mm
- net Net-(R2-Pad2): track 0.00 -> 0.83 mm

Commit message: Renamed Ref
Parts:
- removed 1.25U_PN2, 1.25U_R_ALT1: MX-NoLED, MX_Only:MXOnly-1.25U-Hotswap
- removed 1U_PN1, 1U_R_ALT1, BACKSPLIT1, BACKSPLIT2, DOWNARROW1, FN1, KY_0, KY_1, KY_2, KY_3, KY_4, KY_5, KY_6, KY_7, KY_8, KY_9, KY_A1, KY_B1, KY_C1, KY_COLON1, KY_COMMA1, KY_D1, KY_E1, KY_EQUALS1, KY_ESC1, KY_F1, KY_G1, KY_GRAVE1, KY_H1, KY_I1, KY_J1, KY_K1, KY_L1, KY_LBRACK1, KY_M1, KY_MINUS1, KY_N1, KY_O1, KY_P1, KY_PERIOD1, KY_Q1, KY_QUESTION1: MX-NoLED, MX_Only:MXOnly-1U-Hotswap
- removed 2.75U_SHIFT1: MX-NoLED, MX_Only:MXOnly-2.75U-Hotswap
- removed 2U_BACKSPACE1: MX-NoLED, MX_Only:MXOnly-2U-Hotswap
- removed D1, D10, D11, D12, D13, D14, D15, D16, D17, D18, D19, D2, D20, D21, D22, D23, D24, D25, D26, D27, D28, D29, D3, D30, D31, D32, D33, D34, D35, D36, D37, D38, D39, D4, D40, D41, D42, D43, D44, D45, D46, D47, D48, D49, D5, D50, D51, D52, D53, D54, D55, D56, D57, D58, D59, D6, D60, D61, D62, D63, D64, D65, D66, D67, D7, D8, D9: SOD-123, Diode_SMD:D_SOD-123
- removed F1: 500mA, Fuse:Fuse_1206_3216Metric
- added U2: PRTR5V0U2X, random-keyboard-parts:SOT143B, B.Cu at (200.3, 48.6)
- K19: renamed from MOD_TAB1; value MX-NoLED -> TAB
- K21: renamed from KY_W1; value MX-NoLED -> W
- K23: renamed from KY_R1; value MX-NoLED -> R
- K24: renamed from KY_T1; value MX-NoLED -> T
- K25: renamed from KY_Y1; value MX-NoLED -> Y
- K26: renamed from KY_U1; value MX-NoLED -> U
- K31: renamed from KY_RBRACK1; value MX-NoLED -> }]
- K32: renamed from KY_BAR1; value MX-NoLED -> BAR-BACKSLASH
- K33: renamed from STEPPED_CAPS1; value MX-NoLED -> STEP_CAPS
- K34: renamed from MOD_CAPS1; value MX-NoLED -> CAPS
- K36: renamed from KY_S1; value MX-NoLED -> S
- K45: renamed from KY_QUOTE1; value MX-NoLED -> '
- K46: renamed from MOD_ENTER1; value MX-NoLED -> ENTER
- K47: renamed from MOD_L_SHIFT1; value MX-NoLED -> L_SHIFT
- K48: renamed from KY_Z1; value MX-NoLED -> Z
- K49: renamed from KY_X1; value MX-NoLED -> X
- K51: renamed from KY_V1; value MX-NoLED -> V
- K58: renamed from MOD_R_SHIFT1; value MX-NoLED -> R_SHIFT_1.75U
- K60: renamed from UPARROW1; value MX-NoLED -> UP
- K62: renamed from L_CTRL1; value MX-NoLED -> L_CTRL
- K63: renamed from L_GUI1; value MX-NoLED -> L_GUI
- K64: renamed from L_ALT1; value MX-NoLED -> L_ALT
- K65: renamed from SPACE1; value MX-NoLED -> SPACE
- K70: renamed from R_CTRL1; value MX-NoLED -> R_CTRL
- K71: renamed from LEFTARROW1; value MX-NoLED -> LEFT
- K73: renamed from RIGHTARROW1; value MX-NoLED -> RIGHT
- R6: value 1k -> 10k
- moved R5 198.8 mm to (329.6, 121.7)
- moved R4 61.4 mm to (200.7, 58.4)
- moved R3 57.5 mm to (198.2, 58.4)
- moved K58 52.3 mm to (288.8, 133.9)
- moved K31 52.3 mm to (300.7, 95.8)
- moved K32 52.3 mm to (324.5, 95.8)
- moved K46 52.3 mm to (312.6, 114.9)
- moved K51 52.3 mm to (148.3, 133.9)
- moved K71 52.3 mm to (295.9, 153.0)
- moved R6 52.3 mm to (197.5, 153.8)
- moved R7 52.3 mm to (334.5, 108.5)
- moved Y1 52.3 mm to (205.4, 165.7)
- moved K47 52.3 mm to (60.2, 133.9)
- moved K48 52.3 mm to (91.1, 133.9)
- moved K49 52.3 mm to (110.2, 133.9)
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Routing:
- net Net-(R2-Pad2): track 0.83 -> 0.00 mm

Commit message: Various Fixes
Parts:
- moved K65 89.9 mm to (173.8, 133.3)
- moved K64 34.1 mm to (102.4, 133.3)
- moved K63 27.8 mm to (78.6, 133.3)
- moved K47 20.1 mm to (64.3, 114.3)
- moved K48 20.1 mm to (95.2, 114.3)
- moved K49 20.1 mm to (114.3, 114.3)
- moved K51 20.1 mm to (152.4, 114.3)
- moved K58 20.1 mm to (292.9, 114.3)
- moved K60 20.1 mm to (319.1, 114.3)
- moved USB1 20.1 mm to (203.9, 18.9)
- moved R3 20.1 mm to (202.4, 38.8)
- moved R4 20.1 mm to (204.8, 38.8)
- moved K34 20.1 mm to (69.1, 95.2), turned to 180 degrees
- moved R1 20.1 mm to (206.6, 23.6)
- moved R2 20.1 mm to (200.9, 23.6)
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